Commit message: depth cam updates

File: assets/xacro/panda.mujoco.xacro (robot description, xacro)
@@ -1,4 +1,5 @@
 <?xml version="1.0"?>
 <mujoco xmlns:xacro="http://ros.org/wiki/xacro">
+    <xacro:include filename="panda_camera.mujoco.xacro"/>
     <xacro:if value="${not panda_shared_definitions_loaded}">
         <xacro:property name="panda_shared_definitions_loaded" value="true" />
@@ -101,5 +102,129 @@
     </xacro:if>
     <xacro:macro name="panda_robot" params="name pos rot">
-        <body name="${name}_link0" childclass="panda_robot" pos="${pos}" euler="${rot}"><inertial pos="-0.041018 -0.00014 0.049974" mass="0.629769" fullinertia="0.00315 0.00388 0.004285 8.2904E-07 0.00015 8.2299E-06" /><geom class="panda_robot_visual" mesh="panda_link0_0_visual" material="panda_off_white" /><geom class="panda_robot_visual" mesh="panda_link0_1_visual" material="panda_black" /><geom class="panda_robot_visual" mesh="panda_link0_2_visual" material="panda_off_white" /><geom class="panda_robot_visual" mesh="panda_link0_3_visual" material="panda_black" /><geom class="panda_robot_visual" mesh="panda_link0_4_visual" material="panda_off_white" /><geom class="panda_robot_visual" mesh="panda_link0_5_visual" material="panda_black" /><geom class="panda_robot_visual" mesh="panda_link0_7_visual" material="panda_white" /><geom class="panda_robot_visual" mesh="panda_link0_8_visual" material="panda_white" /><geom class="panda_robot_visual" mesh="panda_link0_9_visual" material="panda_black" /><geom class="panda_robot_visual" mesh="panda_link0_10_visual" material="panda_off_white" /><geom class="panda_robot_visual" mesh="panda_link0_11_visual" material="panda_white" /><geom class="panda_robot_collision" mesh="panda_link0_collision" /><body name="${name}_link1" pos="0 0 0.333"><inertial pos="3.875e-03 2.081e-03 -4.762e-02" mass="4.970684" fullinertia="7.0337e-01 7.0661e-01 9.1170e-03 -1.3900e-04 6.7720e-03 1.9169e-02" /><joint name="${name}_joint1" range="-2.9671 2.9671" /><geom class="panda_robot_visual" mesh="panda_link1_visual" material="panda_white" /><geom class="panda_robot_collision" mesh="panda_link1_collision" /><body name="${name}_link2" pos="0 0 0" quat="0.707107 -0.707107 0 0"><inertial pos="-3.141e-03 -2.872e-02  3.495e-03" mass="0.646926" fullinertia="7.9620e-03 2.8110e-02 2.5995e-02 -3.9250e-03 1.0254e-02 7.0400e-04" /><joint name="${name}_joint2" range="-1.8326 1.8326" /><geom class="panda_robot_visual" mesh="panda_link2_visual" material="panda_white" /><geom class="panda_robot_collision" mesh="panda_link2_collision" /><body name="${name}_link3" pos="0 -0.316 0" quat="0.707107 0.707107 0 0"><inertial pos="2.7518e-02 3.9252e-02 -6.6502e-02" mass="3.228604" fullinertia="3.7242e-02 3.6155e-02 1.0830e-02 -4.7610e-03 -1.1396e-02 -1.2805e-02" /><joint name="${name}_joint3" range="-2.9671 2.9671" /><geom class="panda_robot_visual" mesh="panda_link3_0_visual" material="panda_white" /><geom class="panda_robot_visual" mesh="panda_link3_1_visual" material="panda_white" /><geom class="panda_robot_visual" mesh="panda_link3_2_visual" material="panda_white" /><geom class="panda_robot_visual" mesh="panda_link3_3_visual" material="panda_black" /><geom class="panda_robot_collision" mesh="panda_link3_collision" /><body name="${name}_link4" pos="0.0825 0 0" quat="0.707107 0.707107 0 0"><inertial pos="-5.317e-02 1.04419e-01 2.7454e-02" mass="3.587895" fullinertia="2.5853e-02 1.9552e-02 2.8323e-02 7.7960e-03 -1.3320e-03 8.6410e-03" /><joint name="${name}_joint4" range="-3.1416 -0.4" /><geom class="panda_robot_visual" mesh="panda_link4_0_visual" material="panda_white" /><geom class="panda_robot_visual" mesh="panda_link4_1_visual" material="panda_white" /><geom class="panda_robot_visual" mesh="panda_link4_2_visual" material="panda_black" /><geom class="panda_robot_visual" mesh="panda_link4_3_visual" material="panda_white" /><geom class="panda_robot_collision" mesh="panda_link4_collision" /><body name="${name}_link5" pos="-0.0825 0.384 0" quat="0.707107 -0.707107 0 0"><inertial pos="-1.1953e-02 4.1065e-02 -3.8437e-02" mass="1.225946" fullinertia="3.5549e-02 2.9474e-02 8.6270e-03 -2.1170e-03 -4.0370e-03 2.2900e-04" /><joint name="${name}_joint5" range="-2.9671 2.9671" /><geom class="panda_robot_visual" mesh="panda_link5_0_visual" material="panda_black" /><geom class="panda_robot_visual" mesh="panda_link5_1_visual" material="panda_white" /><geom class="panda_robot_visual" mesh="panda_link5_2_visual" material="panda_white" /><geom class="panda_robot_collision" mesh="panda_link5_0_collision" /><geom class="panda_robot_collision" mesh="panda_link5_1_collision" /><geom class="panda_robot_collision" mesh="panda_link5_2_collision" /><body name="${name}_link6" pos="0 0 0" quat="0.707107 0.707107 0 0"><inertial pos="6.0149e-02 -1.4117e-02 -1.0517e-02" mass="1.666555" fullinertia="1.9640e-03 4.3540e-03 5.4330e-03 1.0900e-04 -1.1580e-03 3.4100e-04" /><joint name="${name}_joint6" range="-0.0873 3.8223" /><geom class="panda_robot_visual" mesh="panda_link6_0_visual" material="panda_off_white" /><geom class="panda_robot_visual" mesh="panda_link6_1_visual" material="panda_white" /><geom class="panda_robot_visual" mesh="panda_link6_2_visual" material="panda_black" /><geom class="panda_robot_visual" mesh="panda_link6_3_visual" material="panda_white" /><geom class="panda_robot_visual" mesh="panda_link6_4_visual" material="panda_white" /><geom class="panda_robot_visual" mesh="panda_link6_5_visual" material="panda_white" /><geom class="panda_robot_visual" mesh="panda_link6_6_visual" material="panda_white" /><geom class="panda_robot_visual" mesh="panda_link6_7_visual" material="panda_light_blue" /><geom class="panda_robot_visual" mesh="panda_link6_8_visual" material="panda_light_blue" /><geom class="panda_robot_visual" mesh="panda_link6_9_visual" material="panda_black" /><geom class="panda_robot_visual" mesh="panda_link6_10_visual" material="panda_black" /><geom class="panda_robot_visual" mesh="panda_link6_11_visual" material="panda_white" /><geom class="panda_robot_visual" mesh="panda_link6_12_visual" material="panda_green" /><geom class="panda_robot_visual" mesh="panda_link6_13_visual" material="panda_white" /><geom class="panda_robot_visual" mesh="panda_link6_14_visual" material="panda_black" /><geom class="panda_robot_visual" mesh="panda_link6_15_visual" material="panda_black" /><geom class="panda_robot_visual" mesh="panda_link6_16_visual" material="panda_white" /><geom class="panda_robot_collision" mesh="panda_link6_collision" /><body name="${name}_link7" pos="0.088 0 0" quat="0.707107 0.707107 0 0"><inertial pos="1.0517e-02 -4.252e-03 6.1597e-02" mass="7.35522e-01" fullinertia="1.2516e-02 1.0027e-02 4.8150e-03 -4.2800e-04 -1.1960e-03 -7.4100e-04" /><joint name="${name}_joint7" range="-2.9671 2.9671" /><geom class="panda_robot_visual" mesh="panda_link7_0_visual" material="panda_white" /><geom class="panda_robot_visual" mesh="panda_link7_1_visual" material="panda_black" /><geom class="panda_robot_visual" mesh="panda_link7_2_visual" material="panda_black" /><geom class="panda_robot_visual" mesh="panda_link7_3_visual" material="panda_black" /><geom class="panda_robot_visual" mesh="panda_link7_4_visual" material="panda_black" /><geom class="panda_robot_visual" mesh="panda_link7_5_visual" material="panda_black" /><geom class="panda_robot_visual" mesh="panda_link7_6_visual" material="panda_black" /><geom class="panda_robot_visual" mesh="panda_link7_7_visual" material="panda_white" /><geom class="panda_robot_collision" mesh="panda_link7_collision" /><body name="${name}_hand" pos="0 0 0.107" quat="0.924  0.0  0.0 -0.383"><inertial pos="-0.01 0 0.03" mass="0.73" diaginertia="0.001 0.0025 0.0017" /><geom class="panda_robot_visual" mesh="panda_hand_0_visual" material="panda_off_white" /><geom class="panda_robot_visual" mesh="panda_hand_1_visual" material="panda_black" /><geom class="panda_robot_visual" mesh="panda_hand_2_visual" material="panda_black" /><geom class="panda_robot_visual" mesh="panda_hand_3_visual" material="panda_white" /><geom class="panda_robot_visual" mesh="panda_hand_4_visual" material="panda_off_white" /><geom class="panda_robot_collision" mesh="panda_hand_collision" /><site name='${name}_ee_site' pos='0 0 0.0' size="0.005 0.005 0.005" euler='0 0 0' /><body name="${name}_leftfinger" pos="0 0 0.0584"><inertial mass="0.015" pos="0 0 0" diaginertia="2.375e-6 2.375e-6 7.5e-7" /><joint class="panda_robot_finger" name="${name}_finger_joint1" axis="0 1 0" type="slide" range="0 0.04" /><geom class="panda_robot_visual" mesh="panda_finger_0_visual" material="panda_off_white" /><geom class="panda_robot_visual" mesh="panda_finger_1_visual" material="panda_black" /><geom class="panda_robot_collision" mesh="panda_finger_0_visual" /><geom class="panda_robot_fingertip_pad_collision_1" /><geom class="panda_robot_fingertip_pad_collision_2" /><geom class="panda_robot_fingertip_pad_collision_3" /><geom class="panda_robot_fingertip_pad_collision_4" /><geom class="panda_robot_fingertip_pad_collision_5" /></body><body name="${name}_rightfinger" pos="0 0 0.0584" quat="0 0 0 1"><inertial mass="0.015" pos="0 0 0" diaginertia="2.375e-6 2.375e-6 7.5e-7" /><joint class="panda_robot_finger" name="${name}_finger_joint2" axis="0 1 0" type="slide" range="0 0.04" /><geom class="panda_robot_visual" mesh="panda_finger_0_visual" material="panda_off_white" /><geom class="panda_robot_visual" mesh="panda_finger_1_visual" material="panda_black" /><geom class="panda_robot_collision" mesh="panda_finger_0_visual" /><geom class="panda_robot_fingertip_pad_collision_1" /><geom class="panda_robot_fingertip_pad_collision_2" /><geom class="panda_robot_fingertip_pad_collision_3" /><geom class="panda_robot_fingertip_pad_collision_4" /><geom class="panda_robot_fingertip_pad_collision_5" /></body></body></body></body></body></body></body></body></body></body>
+        <body name="${name}_link0" childclass="panda_robot" pos="${pos}" euler="${rot}">
+        <inertial pos="-0.041018 -0.00014 0.049974" mass="0.629769" fullinertia="0.00315 0.00388 0.004285 8.2904E-07 0.00015 8.2299E-06" />
+        <geom class="panda_robot_visual" mesh="panda_link0_0_visual" material="panda_off_white" />
+        <geom class="panda_robot_visual" mesh="panda_link0_1_visual" material="panda_black" />
+        <geom class="panda_robot_visual" mesh="panda_link0_2_visual" material="panda_off_white" />
+        <geom class="panda_robot_visual" mesh="panda_link0_3_visual" material="panda_black" />
+        <geom class="panda_robot_visual" mesh="panda_link0_4_visual" material="panda_off_white" />
+        <geom class="panda_robot_visual" mesh="panda_link0_5_visual" material="panda_black" />
+        <geom class="panda_robot_visual" mesh="panda_link0_7_visual" material="panda_white" />
+        <geom class="panda_robot_visual" mesh="panda_link0_8_visual" material="panda_white" />
+        <geom class="panda_robot_visual" mesh="panda_link0_9_visual" material="panda_black" />
+        <geom class="panda_robot_visual" mesh="panda_link0_10_visual" material="panda_off_white" />
+        <geom class="panda_robot_visual" mesh="panda_link0_11_visual" material="panda_white" />
+        <geom class="panda_robot_collision" mesh="panda_link0_collision" />
+        <body name="${name}_link1" pos="0 0 0.333">
+            <inertial pos="3.875e-03 2.081e-03 -4.762e-02" mass="4.970684" fullinertia="7.0337e-01 7.0661e-01 9.1170e-03 -1.3900e-04 6.7720e-03 1.9169e-02" />
+            <joint name="${name}_joint1" range="-2.9671 2.9671" />
+            <geom class="panda_robot_visual" mesh="panda_link1_visual" material="panda_white" />
+            <geom class="panda_robot_collision" mesh="panda_link1_collision" />
+            <body name="${name}_link2" pos="0 0 0" quat="0.707107 -0.707107 0 0">
+                <inertial pos="-3.141e-03 -2.872e-02  3.495e-03" mass="0.646926" fullinertia="7.9620e-03 2.8110e-02 2.5995e-02 -3.9250e-03 1.0254e-02 7.0400e-04" />
+                <joint name="${name}_joint2" range="-1.8326 1.8326" />
+                <geom class="panda_robot_visual" mesh="panda_link2_visual" material="panda_white" />
+                <geom class="panda_robot_collision" mesh="panda_link2_collision" />
+                <body name="${name}_link3" pos="0 -0.316 0" quat="0.707107 0.707107 0 0">
+                    <inertial pos="2.7518e-02 3.9252e-02 -6.6502e-02" mass="3.228604" fullinertia="3.7242e-02 3.6155e-02 1.0830e-02 -4.7610e-03 -1.1396e-02 -1.2805e-02" />
+                    <joint name="${name}_joint3" range="-2.9671 2.9671" />
+                    <geom class="panda_robot_visual" mesh="panda_link3_0_visual" material="panda_white" />
+                    <geom class="panda_robot_visual" mesh="panda_link3_1_visual" material="panda_white" />
+                    <geom class="panda_robot_visual" mesh="panda_link3_2_visual" material="panda_white" />
+                    <geom class="panda_robot_visual" mesh="panda_link3_3_visual" material="panda_black" />
+                    <geom class="panda_robot_collision" mesh="panda_link3_collision" />
+                    <body name="${name}_link4" pos="0.0825 0 0" quat="0.707107 0.707107 0 0">
+                        <inertial pos="-5.317e-02 1.04419e-01 2.7454e-02" mass="3.587895" fullinertia="2.5853e-02 1.9552e-02 2.8323e-02 7.7960e-03 -1.3320e-03 8.6410e-03" />
+                        <joint name="${name}_joint4" range="-3.1416 -0.4" />
+                        <geom class="panda_robot_visual" mesh="panda_link4_0_visual" material="panda_white" />
+                        <geom class="panda_robot_visual" mesh="panda_link4_1_visual" material="panda_white" />
+                        <geom class="panda_robot_visual" mesh="panda_link4_2_visual" material="panda_black" />
+                        <geom class="panda_robot_visual" mesh="panda_link4_3_visual" material="panda_white" />
+                        <geom class="panda_robot_collision" mesh="panda_link4_collision" />
+                        <body name="${name}_link5" pos="-0.0825 0.384 0" quat="0.707107 -0.707107 0 0">
+                            <inertial pos="-1.1953e-02 4.1065e-02 -3.8437e-02" mass="1.225946" fullinertia="3.5549e-02 2.9474e-02 8.6270e-03 -2.1170e-03 -4.0370e-03 2.2900e-04" />
+                            <joint name="${name}_joint5" range="-2.9671 2.9671" />
+                            <geom class="panda_robot_visual" mesh="panda_link5_0_visual" material="panda_black" />
+                            <geom class="panda_robot_visual" mesh="panda_link5_1_visual" material="panda_white" />
+                            <geom class="panda_robot_visual" mesh="panda_link5_2_visual" material="panda_white" />
+                            <geom class="panda_robot_collision" mesh="panda_link5_0_collision" />
+                            <geom class="panda_robot_collision" mesh="panda_link5_1_collision" />
+                            <geom class="panda_robot_collision" mesh="panda_link5_2_collision" />
+                            <body name="${name}_link6" pos="0 0 0" quat="0.707107 0.707107 0 0">
+                                <inertial pos="6.0149e-02 -1.4117e-02 -1.0517e-02" mass="1.666555" fullinertia="1.9640e-03 4.3540e-03 5.4330e-03 1.0900e-04 -1.1580e-03 3.4100e-04" />
+                                <joint name="${name}_joint6" range="-0.0873 3.8223" />
+                                <geom class="panda_robot_visual" mesh="panda_link6_0_visual" material="panda_off_white" />
+                                <geom class="panda_robot_visual" mesh="panda_link6_1_visual" material="panda_white" />
+                                <geom class="panda_robot_visual" mesh="panda_link6_2_visual" material="panda_black" />
+                                <geom class="panda_robot_visual" mesh="panda_link6_3_visual" material="panda_white" />
+                                <geom class="panda_robot_visual" mesh="panda_link6_4_visual" material="panda_white" />
+                                <geom class="panda_robot_visual" mesh="panda_link6_5_visual" material="panda_white" />
+                                <geom class="panda_robot_visual" mesh="panda_link6_6_visual" material="panda_white" />
+                                <geom class="panda_robot_visual" mesh="panda_link6_7_visual" material="panda_light_blue" />
+                                <geom class="panda_robot_visual" mesh="panda_link6_8_visual" material="panda_light_blue" />
+                                <geom class="panda_robot_visual" mesh="panda_link6_9_visual" material="panda_black" />
+                                <geom class="panda_robot_visual" mesh="panda_link6_10_visual" material="panda_black" />
+                                <geom class="panda_robot_visual" mesh="panda_link6_11_visual" material="panda_white" />
+                                <geom class="panda_robot_visual" mesh="panda_link6_12_visual" material="panda_green" />
+                                <geom class="panda_robot_visual" mesh="panda_link6_13_visual" material="panda_white" />
+                                <geom class="panda_robot_visual" mesh="panda_link6_14_visual" material="panda_black" />
+                                <geom class="panda_robot_visual" mesh="panda_link6_15_visual" material="panda_black" />
+                                <geom class="panda_robot_visual" mesh="panda_link6_16_visual" material="panda_white" />
+                                <geom class="panda_robot_collision" mesh="panda_link6_collision" />
+                                <body name="${name}_link7" pos="0.088 0 0" quat="0.707107 0.707107 0 0">
+                                    <inertial pos="1.0517e-02 -4.252e-03 6.1597e-02" mass="7.35522e-01" fullinertia="1.2516e-02 1.0027e-02 4.8150e-03 -4.2800e-04 -1.1960e-03 -7.4100e-04" />
+                                    <joint name="${name}_joint7" range="-2.9671 2.9671" />
+                                    <geom class="panda_robot_visual" mesh="panda_link7_0_visual" material="panda_white" />
+                                    <geom class="panda_robot_visual" mesh="panda_link7_1_visual" material="panda_black" />
+                                    <geom class="panda_robot_visual" mesh="panda_link7_2_visual" material="panda_black" />
+                                    <geom class="panda_robot_visual" mesh="panda_link7_3_visual" material="panda_black" />
+                                    <geom class="panda_robot_visual" mesh="panda_link7_4_visual" material="panda_black" />
+                                    <geom class="panda_robot_visual" mesh="panda_link7_5_visual" material="panda_black" />
+                                    <geom class="panda_robot_visual" mesh="panda_link7_6_visual" material="panda_black" />
+                                    <geom class="panda_robot_visual" mesh="panda_link7_7_visual" material="panda_white" />
+                                    <geom class="panda_robot_collision" mesh="panda_link7_collision" />
+                                    <xacro:panda_camera name="${name}" pos="0.1 -0.1 0.1159" quat="0.924  0.0  0.0 -0.383"/>
+                                    <!-- <body name="${name}_hand" pos="0 0 0.107" quat="0.924  0.0  0.0 -0.383">
+                                        <inertial pos="-0.01 0 0.03" mass="0.73" diaginertia="0.001 0.0025 0.0017" />
+                                        <geom class="panda_robot_visual" mesh="panda_hand_0_visual" material="panda_off_white" />
+                                        <geom class="panda_robot_visual" mesh="panda_hand_1_visual" material="panda_black" />
+                                        <geom class="panda_robot_visual" mesh="panda_hand_2_visual" material="panda_black" />
+                                        <geom class="panda_robot_visual" mesh="panda_hand_3_visual" material="panda_white" />
+                                        <geom class="panda_robot_visual" mesh="panda_hand_4_visual" material="panda_off_white" />
+                                        <geom class="panda_robot_collision" mesh="panda_hand_collision" />
+                                        <site name='${name}_ee_site' pos='0 0 0.0' size="0.005 0.005 0.005" euler='0 0 0' />
+                                            <body name="${name}_leftfinger" pos="0 0 0.0584">
+                                                <inertial mass="0.015" pos="0 0 0" diaginertia="2.375e-6 2.375e-6 7.5e-7" />
+                                                <joint class="panda_robot_finger" name="${name}_finger_joint1" axis="0 1 0" type="slide" range="0 0.04" />
+                                                <geom class="panda_robot_visual" mesh="panda_finger_0_visual" material="panda_off_white" />
+                                                <geom class="panda_robot_visual" mesh="panda_finger_1_visual" material="panda_black" />
+                                                <geom class="panda_robot_collision" mesh="panda_finger_0_visual" />
+                                                <geom class="panda_robot_fingertip_pad_collision_1" />
+                                                <geom class="panda_robot_fingertip_pad_collision_2" />
+                                                <geom class="panda_robot_fingertip_pad_collision_3" />
+                                                <geom class="panda_robot_fingertip_pad_collision_4" />
+                                                <geom class="panda_robot_fingertip_pad_collision_5" />
+                                            </body>
+                                            <body name="${name}_rightfinger" pos="0 0 0.0584" quat="0 0 0 1">
+                                                <inertial mass="0.015" pos="0 0 0" diaginertia="2.375e-6 2.375e-6 7.5e-7" />
+                                                <joint class="panda_robot_finger" name="${name}_finger_joint2" axis="0 1 0" type="slide" range="0 0.04" />
+                                                <geom class="panda_robot_visual" mesh="panda_finger_0_visual" material="panda_off_white" />
+                                                <geom class="panda_robot_visual" mesh="panda_finger_1_visual" material="panda_black" />
+                                                <geom class="panda_robot_collision" mesh="panda_finger_0_visual" />
+                                                <geom class="panda_robot_fingertip_pad_collision_1" />
+                                                <geom class="panda_robot_fingertip_pad_collision_2" />
+                                                <geom class="panda_robot_fingertip_pad_collision_3" />
+                                                <geom class="panda_robot_fingertip_pad_collision_4" />
+                                                <geom class="panda_robot_fingertip_pad_collision_5" />
+                                            </body>
+                                        </body>
+                                    </body> -->
+                                </body>
+                            </body>
+                        </body>
+                    </body>
+                </body>
+            </body>
+        </body>
     </xacro:macro>
     <xacro:macro name="panda_extra" params="name">
