Commit message: camera link fixes

File: assets/xacro/panda.mujoco.xacro (robot description, xacro)
@@ -1,5 +1,4 @@
 <?xml version="1.0"?>
 <mujoco xmlns:xacro="http://ros.org/wiki/xacro">
-    <xacro:include filename="panda_camera.mujoco.xacro"/>
     <xacro:if value="${not panda_shared_definitions_loaded}">
         <xacro:property name="panda_shared_definitions_loaded" value="true" />
@@ -184,5 +183,16 @@
                                     <geom class="panda_robot_visual" mesh="panda_link7_7_visual" material="panda_white" />
                                     <geom class="panda_robot_collision" mesh="panda_link7_collision" />
-                                    <xacro:panda_camera name="${name}" pos="0.05 0.0 0.1159" quat="0.924  0.0  0.0 -0.383"/>
+                                    <body name="${name}_camera_link_fix" pos="0.05 0.0 0.1159" quat="0.92388 0 0 -0.38268">
+                                        <body name="${name}_camera_link" pos="0 0 0" quat="0 0.707107 0 0.707107">
+                                            <geom name="${name}_camera_visual" type="box" size="0.0125 0.045 0.0125" rgba="1 0 0 1" group="2" contype="0" conaffinity="0"/>
+                                            <geom name="${name}_camera_collision" type="box" size="0.0125 0.045 0.0125" rgba="0 0 0 0" group="3"/>
+                                            <inertial pos="0 0 0" mass="0.095" fullinertia="0.0001 0.0001 0.0001 0 0 0" />
+                                            <camera name="${name}_camera" mode="fixed" pos="0 0 0" quat="0.5 -0.5 0.5 -0.5" fovy="70.866"/>
+                                            <body name="${name}_camera_depth_frame" pos="0 0 0" quat="0.5 -0.5 0.5 -0.5">
+                                                <site name="${name}_camera_depth_site" pos="0 0 0" size="0.005 0.005 0.005" euler="0 0 0"/>
+                                            </body>
+                                            <body name="${name}_camera_color_frame" pos="0 0 0" quat="0.5 -0.5 0.5 -0.5"/>
+                                        </body>
+                                    </body>
                                     <body name="${name}_hand" pos="0 0 0.107" quat="0.924  0.0  0.0 -0.383">
                                         <inertial pos="-0.01 0 0.03" mass="0.73" diaginertia="0.001 0.0025 0.0017" />

File: assets/xacro/panda_camera.mujoco.xacro (robot description, xacro)
@@ -1,7 +1,11 @@
 <mujoco xmlns:xacro="http://ros.org/wiki/xacro">
-  <xacro:macro name="panda_camera" params="name pos:='0 0 0.1159' quat:='0.70710678 0 0.70710678 0'">
-    <body name="${name}_camera" pos="${pos}" quat="${quat}">
-      <geom type="box" size="0.0125 0.045 0.0125" rgba="0.5 0.5 0.5 1"/>
-      <camera name="${name}_camera" mode="fixed" pos="0 0 0" fovy="87"/>
+  <xacro:macro name="panda_camera" params="name pos:='0 0 0' euler:='180 -90 0'">
+    <body name="${name}_camera_link_mj" pos="${pos}" euler="${euler}">
+      <geom name="${name}_camera_visual" type="box" size="0.0125 0.045 0.0125" rgba="1 0 0 1" group="2" contype="0" conaffinity="0"/>
+      <geom name="${name}_camera_collision" type="box" size="0.0125 0.045 0.0125" rgba="0 0 0 0" group="3"/>
+      <inertial pos="0 0 0" mass="0.095" fullinertia="0.0001 0.0001 0.0001 0 0 0" />
+      <camera name="${name}_camera" mode="fixed" pos="0 0 0" euler="-90 0 -90" fovy="87"/>
+      <body name="${name}_camera_depth_frame_mj" pos="0 0 0" euler="-90 0 -90"/>
+      <body name="${name}_camera_color_frame_mj" pos="0 0 0" euler="-90 0 -90"/>
     </body>
   </xacro:macro>

Commit message: depth cam rgb fix

File: assets/xacro/panda.mujoco.xacro (robot description, xacro)
@@ -1,4 +1,5 @@
 <?xml version="1.0"?>
 <mujoco xmlns:xacro="http://ros.org/wiki/xacro">
+    <xacro:include filename="panda_camera.mujoco.xacro"/>
     <xacro:if value="${not panda_shared_definitions_loaded}">
         <xacro:property name="panda_shared_definitions_loaded" value="true" />
@@ -184,14 +185,5 @@
                                     <geom class="panda_robot_collision" mesh="panda_link7_collision" />
                                     <body name="${name}_camera_link_fix" pos="0.05 0.0 0.1159" quat="0.92388 0 0 -0.38268">
-                                        <body name="${name}_camera_link" pos="0 0 0" quat="0 0.707107 0 0.707107">
-                                            <geom name="${name}_camera_visual" type="box" size="0.0125 0.045 0.0125" rgba="1 0 0 1" group="2" contype="0" conaffinity="0"/>
-                                            <geom name="${name}_camera_collision" type="box" size="0.0125 0.045 0.0125" rgba="0 0 0 0" group="3"/>
-                                            <inertial pos="0 0 0" mass="0.095" fullinertia="0.0001 0.0001 0.0001 0 0 0" />
-                                            <camera name="${name}_camera" mode="fixed" pos="0 0 0" quat="0.5 -0.5 0.5 -0.5" fovy="70.866"/>
-                                            <body name="${name}_camera_depth_frame" pos="0 0 0" quat="0.5 -0.5 0.5 -0.5">
-                                                <site name="${name}_camera_depth_site" pos="0 0 0" size="0.005 0.005 0.005" euler="0 0 0"/>
-                                            </body>
-                                            <body name="${name}_camera_color_frame" pos="0 0 0" quat="0.5 -0.5 0.5 -0.5"/>
-                                        </body>
+                                        <xacro:panda_camera name="${name}" />
                                     </body>
                                     <body name="${name}_hand" pos="0 0 0.107" quat="0.924  0.0  0.0 -0.383">

File: assets/xacro/panda_camera.mujoco.xacro (robot description, xacro)
@@ -1,11 +1,13 @@
 <mujoco xmlns:xacro="http://ros.org/wiki/xacro">
-  <xacro:macro name="panda_camera" params="name pos:='0 0 0' euler:='180 -90 0'">
-    <body name="${name}_camera_link_mj" pos="${pos}" euler="${euler}">
-      <geom name="${name}_camera_visual" type="box" size="0.0125 0.045 0.0125" rgba="1 0 0 1" group="2" contype="0" conaffinity="0"/>
-      <geom name="${name}_camera_collision" type="box" size="0.0125 0.045 0.0125" rgba="0 0 0 0" group="3"/>
-      <inertial pos="0 0 0" mass="0.095" fullinertia="0.0001 0.0001 0.0001 0 0 0" />
-      <camera name="${name}_camera" mode="fixed" pos="0 0 0" euler="-90 0 -90" fovy="87"/>
-      <body name="${name}_camera_depth_frame_mj" pos="0 0 0" euler="-90 0 -90"/>
-      <body name="${name}_camera_color_frame_mj" pos="0 0 0" euler="-90 0 -90"/>
+  <xacro:macro name="panda_camera" params="name pos:='0 0 0' quat:='0 0.707107 0 0.707107'">
+    <body name="${name}_camera_link" pos="${pos}" quat="${quat}">
+        <geom name="${name}_camera_visual" type="box" size="0.0125 0.045 0.0125" rgba="1 0 0 1" group="2" contype="0" conaffinity="0"/>
+        <geom name="${name}_camera_collision" type="box" size="0.0125 0.045 0.0125" rgba="0 0 0 0" group="3"/>
+        <inertial pos="0 0 0" mass="0.095" fullinertia="0.0001 0.0001 0.0001 0 0 0" />
+        <body name="${name}_camera_depth_frame" pos="0 0 0" quat="0.5 -0.5 0.5 -0.5">
+            <site name="${name}_camera_depth_site" pos="0 0 0" size="0.005 0.005 0.005" euler="0 0 0"/>
+            <camera name="${name}_camera" mode="fixed" pos="0 0 0" quat="0 1 0 0" fovy="70.866"/>
+        </body>
+        <body name="${name}_camera_color_frame" pos="0 0 0" quat="0.5 -0.5 0.5 -0.5"/>
     </body>
   </xacro:macro>
